Commit message: return to REPUSH

File: RCKO2025_description/urdf/RCKO2025.xacro (robot description, xacro)
@@ -146,7 +146,13 @@
 <link name="left_lower_leg_1">
   <inertial>
+<<<<<<< HEAD
     <origin xyz="-0.005650281818702613 0.025822001462742536 -0.06772036929997684" rpy="0 0 0"/>
     <mass value="0.10974623051687926"/>
     <inertia ixx="0.000262" iyy="0.000201" izz="8e-05" ixy="-0.0" iyz="-0.0" ixz="-1.4e-05"/>
+=======
+    <origin xyz="-8.212056945443085e-05 0.02582198317065247 -0.06795536785927819" rpy="0 0 0"/>
+    <mass value="0.1097462305168792"/>
+    <inertia ixx="0.000263" iyy="0.000201" izz="7.9e-05" ixy="0.0" iyz="-0.0" ixz="1e-06"/>
+>>>>>>> parent of 44e5b30 (repush)
   </inertial>
   <visual>
@@ -166,7 +172,13 @@
 <link name="right_lower_leg_1">
   <inertial>
+<<<<<<< HEAD
     <origin xyz="-0.005008387197218772 -0.025566931779343473 -0.0675226987376316" rpy="0 0 0"/>
     <mass value="0.10974623051688356"/>
     <inertia ixx="0.000262" iyy="0.000201" izz="8e-05" ixy="-0.0" iyz="-1e-06" ixz="-1.2e-05"/>
+=======
+    <origin xyz="0.0005403758644122038 -0.025566943522814516 -0.06770626577304717" rpy="0 0 0"/>
+    <mass value="0.10974623051688351"/>
+    <inertia ixx="0.000263" iyy="0.000201" izz="7.9e-05" ixy="0.0" iyz="-1e-06" ixz="3e-06"/>
+>>>>>>> parent of 44e5b30 (repush)
   </inertial>
   <visual>
@@ -186,7 +198,13 @@
 <link name="left_ankle_pitch_1">
   <inertial>
+<<<<<<< HEAD
     <origin xyz="-0.0012523271413189263 -0.02587212282028315 0.017519682372607585" rpy="0 0 0"/>
     <mass value="0.7617305331247881"/>
     <inertia ixx="0.000377" iyy="0.000355" izz="0.000247" ixy="2e-06" iyz="1e-06" ixz="1.3e-05"/>
+=======
+    <origin xyz="-0.002684447385301289 -0.02587219041070523 0.017358487086665916" rpy="0 0 0"/>
+    <mass value="0.7617305331247872"/>
+    <inertia ixx="0.000374" iyy="0.000355" izz="0.00025" ixy="2e-06" iyz="2e-06" ixz="2.3e-05"/>
+>>>>>>> parent of 44e5b30 (repush)
   </inertial>
   <visual>
@@ -206,7 +224,13 @@
 <link name="right_ankle_pitch_1">
   <inertial>
+<<<<<<< HEAD
     <origin xyz="-0.0009647138858091819 0.026039726449397026 0.017289135778773165" rpy="0 0 0"/>
     <mass value="0.7617304834003347"/>
     <inertia ixx="0.000378" iyy="0.000355" izz="0.000247" ixy="-2e-06" iyz="-2e-06" ixz="1.1e-05"/>
+=======
+    <origin xyz="-0.002677931766474576 0.02603954060499232 0.017107353866920166" rpy="0 0 0"/>
+    <mass value="0.7617304834003356"/>
+    <inertia ixx="0.000375" iyy="0.000355" izz="0.00025" ixy="-1e-06" iyz="-3e-06" ixz="2.3e-05"/>
+>>>>>>> parent of 44e5b30 (repush)
   </inertial>
   <visual>
@@ -330,6 +354,11 @@
   <axis xyz="0.996014 -5e-06 -0.089201"/>
 </joint>
+<<<<<<< HEAD
 <joint name="rotate_20" type="continuous">
   <origin xyz="-0.038898 -0.024169 0.022933" rpy="0 0 0"/>
+=======
+<joint name="ȸ�� 13" type="continuous">
+  <origin xyz="-0.040647 -0.024169 0.019669" rpy="0 0 0"/>
+>>>>>>> parent of 44e5b30 (repush)
   <parent link="left_ankle_pitch_1"/>
   <child link="left_foot_1"/>

Commit message: normal

File: RCKO2025_description/urdf/RCKO2025.xacro (robot description, xacro)
@@ -6,7 +6,7 @@
 <link name="base_link">
   <inertial>
-    <origin xyz="-0.0781198333354195 -0.0006518299308106812 0.4399478846677073" rpy="0 0 0"/>
+    <origin xyz="-0.016297126176947143 0.0025458330031376073 0.46299748907258126" rpy="0 0 0"/>
     <mass value="6.741980845925567"/>
-    <inertia ixx="0.113784" iyy="0.061497" izz="0.065417" ixy="-0.00012" iyz="-0.000837" ixz="-0.008419"/>
+    <inertia ixx="0.114834" iyy="0.061497" izz="0.064366" ixy="-5.1e-05" iyz="-0.000843" ixz="-0.004356"/>
   </inertial>
   <visual>
@@ -26,10 +26,10 @@
 <link name="left_hipjoint_abd_1">
   <inertial>
-    <origin xyz="-0.0596233437641636 -1.5916383786993005e-05 -0.042812233695081636" rpy="0 0 0"/>
+    <origin xyz="-0.05591415809537886 -1.5871339073603163e-05 -0.04755389203614463" rpy="0 0 0"/>
     <mass value="0.6286646646290881"/>
-    <inertia ixx="0.000271" iyy="0.000482" izz="0.000331" ixy="-0.0" iyz="-0.0" ixz="-0.00011"/>
-  </inertial>
-  <visual>
-    <origin xyz="0.070374 -0.04534 -0.356795" rpy="0 0 0"/>
+    <inertia ixx="0.000289" iyy="0.000482" izz="0.000312" ixy="-0.0" iyz="-0.0" ixz="-0.000113"/>
+  </inertial>
+  <visual>
+    <origin xyz="0.001764 -0.048538 -0.380759" rpy="0 0 0"/>
     <geometry>
       <mesh filename="file://$(find RCKO2025_description)/meshes/left_hipjoint_abd_1.stl" scale="0.001 0.001 0.001"/>
@@ -38,5 +38,5 @@
   </visual>
   <collision>
-    <origin xyz="0.070374 -0.04534 -0.356795" rpy="0 0 0"/>
+    <origin xyz="0.001764 -0.048538 -0.380759" rpy="0 0 0"/>
     <geometry>
       <mesh filename="file://$(find RCKO2025_description)/meshes/left_hipjoint_abd_1.stl" scale="0.001 0.001 0.001"/>
@@ -46,10 +46,10 @@
 <link name="right_hipjoint_abd_1">
   <inertial>
-    <origin xyz="-0.05962271764844841 -1.591164752746954e-05 -0.04281225817161166" rpy="0 0 0"/>
+    <origin xyz="-0.05591415817974288 -1.5866569012319698e-05 -0.04755458650877381" rpy="0 0 0"/>
     <mass value="0.6286646646151826"/>
-    <inertia ixx="0.000271" iyy="0.000482" izz="0.000331" ixy="-0.0" iyz="-0.0" ixz="-0.00011"/>
-  </inertial>
-  <visual>
-    <origin xyz="0.070371 0.04466 -0.356824" rpy="0 0 0"/>
+    <inertia ixx="0.000289" iyy="0.000482" izz="0.000312" ixy="-0.0" iyz="-0.0" ixz="-0.000113"/>
+  </inertial>
+  <visual>
+    <origin xyz="0.001764 0.041462 -0.380789" rpy="0 0 0"/>
     <geometry>
       <mesh filename="file://$(find RCKO2025_description)/meshes/right_hipjoint_abd_1.stl" scale="0.001 0.001 0.001"/>
@@ -58,5 +58,5 @@
   </visual>
   <collision>
-    <origin xyz="0.070371 0.04466 -0.356824" rpy="0 0 0"/>
+    <origin xyz="0.001764 0.041462 -0.380789" rpy="0 0 0"/>
     <geometry>
       <mesh filename="file://$(find RCKO2025_description)/meshes/right_hipjoint_abd_1.stl" scale="0.001 0.001 0.001"/>
@@ -66,10 +66,10 @@
 <link name="right_hipjoint_pitch_1">
   <inertial>
-    <origin xyz="0.03795351737590434 -0.0017766974421925888 -0.000954299033687378" rpy="0 0 0"/>
+    <origin xyz="0.0379043656699808 -0.0017774058233399684 0.00215803669318948" rpy="0 0 0"/>
     <mass value="0.7374479075497384"/>
-    <inertia ixx="0.000347" iyy="0.000346" izz="0.000238" ixy="1e-06" iyz="-3e-06" ixz="-3e-05"/>
-  </inertial>
-  <visual>
-    <origin xyz="0.116663 0.044682 -0.293404" rpy="0 0 0"/>
+    <inertia ixx="0.000352" iyy="0.000346" izz="0.000233" ixy="1e-06" iyz="-2e-06" ixz="-2.1e-05"/>
+  </inertial>
+  <visual>
+    <origin xyz="0.042704 0.041484 -0.313789" rpy="0 0 0"/>
     <geometry>
       <mesh filename="file://$(find RCKO2025_description)/meshes/right_hipjoint_pitch_1.stl" scale="0.001 0.001 0.001"/>
@@ -78,5 +78,5 @@
   </visual>
   <collision>
-    <origin xyz="0.116663 0.044682 -0.293404" rpy="0 0 0"/>
+    <origin xyz="0.042704 0.041484 -0.313789" rpy="0 0 0"/>
     <geometry>
       <mesh filename="file://$(find RCKO2025_description)/meshes/right_hipjoint_pitch_1.stl" scale="0.001 0.001 0.001"/>
@@ -86,10 +86,10 @@
 <link name="left_hipjoint_pitch_1">
   <inertial>
-    <origin xyz="0.03795174115874955 0.0017985655564198358 -0.0009715126126632612" rpy="0 0 0"/>
+    <origin xyz="0.03790436613028492 0.0017978502289910728 0.0021413949329527338" rpy="0 0 0"/>
     <mass value="0.7374478792065627"/>
-    <inertia ixx="0.000347" iyy="0.000346" izz="0.000238" ixy="-2e-06" iyz="1e-06" ixz="-3e-05"/>
-  </inertial>
-  <visual>
-    <origin xyz="0.116168 -0.045318 -0.293334" rpy="0 0 0"/>
+    <inertia ixx="0.000352" iyy="0.000346" izz="0.000233" ixy="-2e-06" iyz="1e-06" ixz="-2.1e-05"/>
+  </inertial>
+  <visual>
+    <origin xyz="0.042204 -0.048516 -0.313759" rpy="0 0 0"/>
     <geometry>
       <mesh filename="file://$(find RCKO2025_description)/meshes/left_hipjoint_pitch_1.stl" scale="0.001 0.001 0.001"/>
@@ -98,5 +98,5 @@
   </visual>
   <collision>
-    <origin xyz="0.116168 -0.045318 -0.293334" rpy="0 0 0"/>
+    <origin xyz="0.042204 -0.048516 -0.313759" rpy="0 0 0"/>
     <geometry>
       <mesh filename="file://$(find RCKO2025_description)/meshes/left_hipjoint_pitch_1.stl" scale="0.001 0.001 0.001"/>
@@ -106,10 +106,10 @@
 <link name="right_upper_leg__1">
   <inertial>
-    <origin xyz="-0.0008668984942271918 0.022238946917568732 -0.1149019351658267" rpy="0 0 0"/>
+    <origin xyz="0.008551612660915009 0.022238944873896056 -0.11458656880466644" rpy="0 0 0"/>
     <mass value="0.8327131213392032"/>
-    <inertia ixx="0.001217" iyy="0.00113" izz="0.00036" ixy="-2e-06" iyz="-3e-06" ixz="-0.000114"/>
-  </inertial>
-  <visual>
-    <origin xyz="0.074661 0.068722 -0.310006" rpy="0 0 0"/>
+    <inertia ixx="0.00123" iyy="0.00113" izz="0.000347" ixy="-2e-06" iyz="-4e-06" ixz="-4.2e-05"/>
+  </inertial>
+  <visual>
+    <origin xyz="0.002204 0.065525 -0.333776" rpy="0 0 0"/>
     <geometry>
       <mesh filename="file://$(find RCKO2025_description)/meshes/right_upper_leg__1.stl" scale="0.001 0.001 0.001"/>
@@ -118,5 +118,5 @@
   </visual>
   <collision>
-    <origin xyz="0.074661 0.068722 -0.310006" rpy="0 0 0"/>
+    <origin xyz="0.002204 0.065525 -0.333776" rpy="0 0 0"/>
     <geometry>
       <mesh filename="file://$(find RCKO2025_description)/meshes/right_upper_leg__1.stl" scale="0.001 0.001 0.001"/>
@@ -126,10 +126,10 @@
 <link name="left_upper_leg__1">
   <inertial>
-    <origin xyz="-0.0021618860453990613 -0.023349404547272537 -0.11466448257668885" rpy="0 0 0"/>
+    <origin xyz="0.007241030065429671 -0.02334939560791792 -0.11445621861481967" rpy="0 0 0"/>
     <mass value="0.8327131573768546"/>
-    <inertia ixx="0.001214" iyy="0.00113" izz="0.000363" ixy="1e-06" iyz="-4e-06" ixz="-0.000123"/>
-  </inertial>
-  <visual>
-    <origin xyz="0.074186 -0.069552 -0.309703" rpy="0 0 0"/>
+    <inertia ixx="0.001229" iyy="0.00113" izz="0.000348" ixy="1e-06" iyz="-4e-06" ixz="-5.2e-05"/>
+  </inertial>
+  <visual>
+    <origin xyz="0.001704 -0.072749 -0.333513" rpy="0 0 0"/>
     <geometry>
       <mesh filename="file://$(find RCKO2025_description)/meshes/left_upper_leg__1.stl" scale="0.001 0.001 0.001"/>
@@ -138,5 +138,5 @@
   </visual>
   <collision>
-    <origin xyz="0.074186 -0.069552 -0.309703" rpy="0 0 0"/>
+    <origin xyz="0.001704 -0.072749 -0.333513" rpy="0 0 0"/>
     <geometry>
       <mesh filename="file://$(find RCKO2025_description)/meshes/left_upper_leg__1.stl" scale="0.001 0.001 0.001"/>
@@ -146,10 +146,10 @@
 <link name="left_lower_leg_1">
   <inertial>
-    <origin xyz="-0.005650281818702613 0.025822001462742536 -0.06772036929997684" rpy="0 0 0"/>
+    <origin xyz="-8.212056945443085e-05 0.02582198317065247 -0.06795536785927817" rpy="0 0 0"/>
     <mass value="0.10974623051687926"/>
-    <inertia ixx="0.000262" iyy="0.000201" izz="8e-05" ixy="-0.0" iyz="-0.0" ixz="-1.4e-05"/>
-  </inertial>
-  <visual>
-    <origin xyz="0.086132 0.072592 -0.170487" rpy="0 0 0"/>
+    <inertia ixx="0.000263" iyy="0.000201" izz="7.9e-05" ixy="0.0" iyz="-0.0" ixz="1e-06"/>
+  </inertial>
+  <visual>
+    <origin xyz="0.002204 0.069395 -0.193786" rpy="0 0 0"/>
     <geometry>
       <mesh filename="file://$(find RCKO2025_description)/meshes/left_lower_leg_1.stl" scale="0.001 0.001 0.001"/>
@@ -158,5 +158,5 @@
   </visual>
   <collision>
-    <origin xyz="0.086132 0.072592 -0.170487" rpy="0 0 0"/>
+    <origin xyz="0.002204 0.069395 -0.193786" rpy="0 0 0"/>
     <geometry>
       <mesh filename="file://$(find RCKO2025_description)/meshes/left_lower_leg_1.stl" scale="0.001 0.001 0.001"/>
@@ -166,10 +166,10 @@
 <link name="right_lower_leg_1">
   <inertial>
-    <origin xyz="-0.005008387197218772 -0.025566931779343473 -0.0675226987376316" rpy="0 0 0"/>
+    <origin xyz="0.0005403758644121504 -0.02556694352281455 -0.0677062657730472" rpy="0 0 0"/>
     <mass value="0.10974623051688356"/>
-    <inertia ixx="0.000262" iyy="0.000201" izz="8e-05" ixy="-0.0" iyz="-1e-06" ixz="-1.2e-05"/>
-  </inertial>
-  <visual>
-    <origin xyz="0.087255 -0.072064 -0.170293" rpy="0 0 0"/>
+    <inertia ixx="0.000263" iyy="0.000201" izz="7.9e-05" ixy="0.0" iyz="-1e-06" ixz="3e-06"/>
+  </inertial>
+  <visual>
+    <origin xyz="0.003305 -0.075261 -0.193501" rpy="0 0 0"/>
     <geometry>
       <mesh filename="file://$(find RCKO2025_description)/meshes/right_lower_leg_1.stl" scale="0.001 0.001 0.001"/>
@@ -178,5 +178,5 @@
   </visual>
   <collision>
-    <origin xyz="0.087255 -0.072064 -0.170293" rpy="0 0 0"/>
+    <origin xyz="0.003305 -0.075261 -0.193501" rpy="0 0 0"/>
     <geometry>
       <mesh filename="file://$(find RCKO2025_description)/meshes/right_lower_leg_1.stl" scale="0.001 0.001 0.001"/>
@@ -186,10 +186,10 @@
 <link name="left_ankle_pitch_1">
   <inertial>
-    <origin xyz="-0.0012523271413189263 -0.02587212282028315 0.017519682372607585" rpy="0 0 0"/>
-    <mass value="0.7617305331247881"/>
-    <inertia ixx="0.000377" iyy="0.000355" izz="0.000247" ixy="2e-06" iyz="1e-06" ixz="1.3e-05"/>
-  </inertial>
-  <visual>
-    <origin xyz="0.097226 -0.071989 -0.030646" rpy="0 0 0"/>
+    <origin xyz="-0.0026844530151543702 -0.02587218408919989 0.017358486982995885" rpy="0 0 0"/>
+    <mass value="0.7617305331247886"/>
+    <inertia ixx="0.000374" iyy="0.000355" izz="0.00025" ixy="2e-06" iyz="2e-06" ixz="2.3e-05"/>
+  </inertial>
+  <visual>
+    <origin xyz="0.0018 -0.075186 -0.053506" rpy="0 0 0"/>
     <geometry>
       <mesh filename="file://$(find RCKO2025_description)/meshes/left_ankle_pitch_1.stl" scale="0.001 0.001 0.001"/>
@@ -198,5 +198,5 @@
   </visual>
   <collision>
-    <origin xyz="0.097226 -0.071989 -0.030646" rpy="0 0 0"/>
+    <origin xyz="0.0018 -0.075186 -0.053506" rpy="0 0 0"/>
     <geometry>
       <mesh filename="file://$(find RCKO2025_description)/meshes/left_ankle_pitch_1.stl" scale="0.001 0.001 0.001"/>
@@ -206,10 +206,10 @@
 <link name="right_ankle_pitch_1">
   <inertial>
-    <origin xyz="-0.0009647138858091819 0.026039726449397026 0.017289135778773165" rpy="0 0 0"/>
-    <mass value="0.7617304834003347"/>
-    <inertia ixx="0.000378" iyy="0.000355" izz="0.000247" ixy="-2e-06" iyz="-2e-06" ixz="1.1e-05"/>
-  </inertial>
-  <visual>
-    <origin xyz="0.097384 0.072962 -0.03094" rpy="0 0 0"/>
+    <origin xyz="-0.0023777503230411894 0.026039657267006668 0.01715148217324003" rpy="0 0 0"/>
+    <mass value="0.7617304834003343"/>
+    <inertia ixx="0.000375" iyy="0.000355" izz="0.000249" ixy="-1e-06" iyz="-3e-06" ixz="2.1e-05"/>
+  </inertial>
+  <visual>
+    <origin xyz="0.001984 0.069765 -0.053787" rpy="0 0 0"/>
     <geometry>
       <mesh filename="file://$(find RCKO2025_description)/meshes/right_ankle_pitch_1.stl" scale="0.001 0.001 0.001"/>
@@ -218,5 +218,5 @@
   </visual>
   <collision>
-    <origin xyz="0.097384 0.072962 -0.03094" rpy="0 0 0"/>
+    <origin xyz="0.001984 0.069765 -0.053787" rpy="0 0 0"/>
     <geometry>
       <mesh filename="file://$(find RCKO2025_description)/meshes/right_ankle_pitch_1.stl" scale="0.001 0.001 0.001"/>
@@ -226,10 +226,10 @@
 <link name="right_foot_1">
   <inertial>
-    <origin xyz="0.0014179546955375988 -0.00592191825624204 -0.03650825547499402" rpy="0 0 0"/>
-    <mass value="1.0884519024049495"/>
-    <inertia ixx="0.001325" iyy="0.002955" izz="0.00273" ixy="0.00016" iyz="-0.000159" ixz="0.000749"/>
-  </inertial>
-  <visual>
-    <origin xyz="0.135891 0.048602 -0.054328" rpy="0 0 0"/>
+    <origin xyz="0.004403987733357477 -0.005921573975609225 -0.03626861876211406" rpy="0 0 0"/>
+    <mass value="1.0884519024049497"/>
+    <inertia ixx="0.001212" iyy="0.002955" izz="0.002843" ixy="0.000173" iyz="-0.000146" ixz="0.000624"/>
+  </inertial>
+  <visual>
+    <origin xyz="0.042277 0.045405 -0.07394" rpy="0 0 0"/>
     <geometry>
       <mesh filename="file://$(find RCKO2025_description)/meshes/right_foot_1.stl" scale="0.001 0.001 0.001"/>
@@ -238,5 +238,5 @@
   </visual>
   <collision>
-    <origin xyz="0.135891 0.048602 -0.054328" rpy="0 0 0"/>
+    <origin xyz="0.042277 0.045405 -0.07394" rpy="0 0 0"/>
     <geometry>
       <mesh filename="file://$(find RCKO2025_description)/meshes/right_foot_1.stl" scale="0.001 0.001 0.001"/>
@@ -246,10 +246,10 @@
 <link name="left_foot_1">
   <inertial>
-    <origin xyz="0.0020652511099268356 0.005859471466279832 -0.03648673300507772" rpy="0 0 0"/>
-    <mass value="1.0884519419711154"/>
-    <inertia ixx="0.001299" iyy="0.002955" izz="0.002756" ixy="-0.000162" iyz="0.000156" ixz="0.000724"/>
-  </inertial>
-  <visual>
-    <origin xyz="0.136124 -0.04782 -0.053579" rpy="0 0 0"/>
+    <origin xyz="0.00504798443398731 0.005859814548277609 -0.036194859990575305" rpy="0 0 0"/>
+    <mass value="1.088451941971115"/>
+    <inertia ixx="0.00119" iyy="0.002955" izz="0.002864" ixy="-0.000174" iyz="0.000142" ixz="0.000595"/>
+  </inertial>
+  <visual>
+    <origin xyz="0.042447 -0.051017 -0.073175" rpy="0 0 0"/>
     <geometry>
       <mesh filename="file://$(find RCKO2025_description)/meshes/left_foot_1.stl" scale="0.001 0.001 0.001"/>
@@ -258,5 +258,5 @@
   </visual>
   <collision>
-    <origin xyz="0.136124 -0.04782 -0.053579" rpy="0 0 0"/>
+    <origin xyz="0.042447 -0.051017 -0.073175" rpy="0 0 0"/>
     <geometry>
       <mesh filename="file://$(find RCKO2025_description)/meshes/left_foot_1.stl" scale="0.001 0.001 0.001"/>
@@ -265,74 +265,74 @@
 </link>
 <joint name="rotate_12" type="continuous">
-  <origin xyz="-0.070374 0.04534 0.356795" rpy="0 0 0"/>
+  <origin xyz="-0.001764 0.048538 0.380759" rpy="0 0 0"/>
   <parent link="base_link"/>
   <child link="left_hipjoint_abd_1"/>
-  <axis xyz="-0.081939 -0.000324 -0.996637"/>
+  <axis xyz="-0.0 -0.000326 -1.0"/>
 </joint>
 <joint name="rotate_13" type="continuous">
-  <origin xyz="-0.070371 -0.04466 0.356824" rpy="0 0 0"/>
+  <origin xyz="-0.001764 -0.041462 0.380789" rpy="0 0 0"/>
   <parent link="base_link"/>
   <child link="right_hipjoint_abd_1"/>
-  <axis xyz="-0.081939 -0.000324 -0.996637"/>
+  <axis xyz="-0.0 -0.000326 -1.0"/>
 </joint>
 <joint name="rotate_10" type="continuous">
-  <origin xyz="-0.046292 -2.2e-05 -0.06342" rpy="0 0 0"/>
+  <origin xyz="-0.04094 -2.2e-05 -0.067" rpy="0 0 0"/>
   <parent link="right_hipjoint_abd_1"/>
   <child link="right_hipjoint_pitch_1"/>
-  <axis xyz="0.996637 1.4e-05 -0.081939"/>
+  <axis xyz="1.0 0.0 0.0"/>
 </joint>
 <joint name="rotate_11" type="continuous">
-  <origin xyz="-0.045794 -2.2e-05 -0.063461" rpy="0 0 0"/>
+  <origin xyz="-0.04044 -2.2e-05 -0.067" rpy="0 0 0"/>
   <parent link="left_hipjoint_abd_1"/>
   <child link="left_hipjoint_pitch_1"/>
-  <axis xyz="0.996637 1.4e-05 -0.081939"/>
+  <axis xyz="1.0 -0.0 0.0"/>
 </joint>
 <joint name="rotate_15" type="continuous">
-  <origin xyz="0.042002 -0.02404 0.016602" rpy="0 0 0"/>
+  <origin xyz="0.0405 -0.024041 0.019987" rpy="0 0 0"/>
   <parent link="right_hipjoint_pitch_1"/>
   <child link="right_upper_leg__1"/>
-  <axis xyz="0.00023 -0.999997 0.002632"/>
+  <axis xyz="-0.0 -0.999997 0.002644"/>
 </joint>
 <joint name="rotate_14" type="continuous">
-  <origin xyz="0.041982 0.024234 0.016369" rpy="0 0 0"/>
+  <origin xyz="0.0405 0.024233 0.019754" rpy="0 0 0"/>
   <parent link="left_hipjoint_pitch_1"/>
   <child link="left_upper_leg__1"/>
-  <axis xyz="-0.000592 0.999975 -0.007027"/>
+  <axis xyz="0.0 0.999975 -0.007053"/>
 </joint>
 <joint name="rotate_17" type="continuous">
-  <origin xyz="-0.011471 -0.00387 -0.139519" rpy="0 0 0"/>
+  <origin xyz="0.0 -0.00387 -0.13999" rpy="0 0 0"/>
   <parent link="right_upper_leg__1"/>
   <child link="left_lower_leg_1"/>
-  <axis xyz="0.00023 -0.999997 0.002632"/>
+  <axis xyz="-0.0 -0.999997 0.002644"/>
 </joint>
 <joint name="rotate_16" type="continuous">
-  <origin xyz="-0.013069 0.002512 -0.13941" rpy="0 0 0"/>
+  <origin xyz="-0.001601 0.002512 -0.140012" rpy="0 0 0"/>
   <parent link="left_upper_leg__1"/>
   <child link="right_lower_leg_1"/>
-  <axis xyz="-0.000592 0.999975 -0.007027"/>
+  <axis xyz="0.0 0.999975 -0.007053"/>
 </joint>
 <joint name="rotate_18" type="continuous">
-  <origin xyz="-0.009971 -7.5e-05 -0.139647" rpy="0 0 0"/>
+  <origin xyz="0.001505 -7.5e-05 -0.139995" rpy="0 0 0"/>
   <parent link="right_lower_leg_1"/>
   <child link="left_ankle_pitch_1"/>
-  <axis xyz="0.000592 -0.999975 0.007027"/>
+  <axis xyz="-0.0 -0.999975 0.007053"/>
 </joint>
 <joint name="rotate_19" type="continuous">
-  <origin xyz="-0.011252 -0.00037 -0.139547" rpy="0 0 0"/>
+  <origin xyz="0.00022 -0.00037 -0.139999" rpy="0 0 0"/>
   <parent link="left_lower_leg_1"/>
   <child link="right_ankle_pitch_1"/>
-  <axis xyz="-0.00023 0.999997 -0.002632"/>
+  <axis xyz="0.0 0.999997 -0.002644"/>
 </joint>
 <joint name="rotate_21" type="continuous">
-  <origin xyz="-0.038507 0.02436 0.023388" rpy="0 0 0"/>
+  <origin xyz="-0.040293 0.02436 0.020153" rpy="0 0 0"/>
   <parent link="right_ankle_pitch_1"/>
   <child link="right_foot_1"/>
-  <axis xyz="0.996014 -5e-06 -0.089201"/>
+  <axis xyz="0.999973 -1.9e-05 -0.007289"/>
 </joint>
 <joint name="rotate_20" type="continuous">
-  <origin xyz="-0.038898 -0.024169 0.022933" rpy="0 0 0"/>
+  <origin xyz="-0.040647 -0.024169 0.019669" rpy="0 0 0"/>
   <parent link="left_ankle_pitch_1"/>
   <child link="left_foot_1"/>
-  <axis xyz="0.997442 8.8e-05 -0.071476"/>
+  <axis xyz="0.999945 7.4e-05 0.010493"/>
 </joint>
 </robot>
