Commit message: 512_12DOF

File: RCKO_512_12DOF/robocup_2025_description/urdf/materials.xacro (robot description, xacro)
@@ -1,4 +1,4 @@
 <?xml version="1.0" ?>
-<robot name="RCKO2025" xmlns:xacro="http://www.ros.org/wiki/xacro" >
+<robot name="robocup_2025" xmlns:xacro="http://www.ros.org/wiki/xacro" >
 <material name="silver">
   <color rgba="0.700 0.700 0.700 1.000"/>

File: RCKO_512_12DOF/robocup_2025_description/urdf/robocup_2025.xacro (robot description, xacro)
@@ -1,7 +1,7 @@
 <?xml version="1.0" ?>
-<robot name="RCKO2025" xmlns:xacro="http://www.ros.org/wiki/xacro">
-<xacro:include filename="$(find RCKO2025_description)/urdf/materials.xacro" />
-<xacro:include filename="$(find RCKO2025_description)/urdf/RCKO2025.trans" />
-<xacro:include filename="$(find RCKO2025_description)/urdf/RCKO2025.gazebo" />
+<robot name="robocup_2025" xmlns:xacro="http://www.ros.org/wiki/xacro">
+<xacro:include filename="$(find robocup_2025_description)/urdf/materials.xacro" />
+<xacro:include filename="$(find robocup_2025_description)/urdf/robocup_2025.trans" />
+<xacro:include filename="$(find robocup_2025_description)/urdf/robocup_2025.gazebo" />
 <link name="base_link">
   <inertial>
@@ -13,5 +13,5 @@
     <origin xyz="0 0 0" rpy="0 0 0"/>
     <geometry>
-      <mesh filename="file://$(find RCKO2025_description)/meshes/base_link.stl" scale="0.001 0.001 0.001"/>
+      <mesh filename="file://$(find robocup_2025_description)/meshes/base_link.stl" scale="0.001 0.001 0.001"/>
     </geometry>
     <material name="silver"/>
@@ -20,5 +20,5 @@
     <origin xyz="0 0 0" rpy="0 0 0"/>
     <geometry>
-      <mesh filename="file://$(find RCKO2025_description)/meshes/base_link.stl" scale="0.001 0.001 0.001"/>
+      <mesh filename="file://$(find robocup_2025_description)/meshes/base_link.stl" scale="0.001 0.001 0.001"/>
     </geometry>
   </collision>
@@ -33,5 +33,5 @@
     <origin xyz="0.001764 -0.048538 -0.380759" rpy="0 0 0"/>
     <geometry>
-      <mesh filename="file://$(find RCKO2025_description)/meshes/left_hipjoint_abd_1.stl" scale="0.001 0.001 0.001"/>
+      <mesh filename="file://$(find robocup_2025_description)/meshes/left_hipjoint_abd_1.stl" scale="0.001 0.001 0.001"/>
     </geometry>
     <material name="silver"/>
@@ -40,5 +40,5 @@
     <origin xyz="0.001764 -0.048538 -0.380759" rpy="0 0 0"/>
     <geometry>
-      <mesh filename="file://$(find RCKO2025_description)/meshes/left_hipjoint_abd_1.stl" scale="0.001 0.001 0.001"/>
+      <mesh filename="file://$(find robocup_2025_description)/meshes/left_hipjoint_abd_1.stl" scale="0.001 0.001 0.001"/>
     </geometry>
   </collision>
@@ -53,5 +53,5 @@
     <origin xyz="0.001764 0.041462 -0.380789" rpy="0 0 0"/>
     <geometry>
-      <mesh filename="file://$(find RCKO2025_description)/meshes/right_hipjoint_abd_1.stl" scale="0.001 0.001 0.001"/>
+      <mesh filename="file://$(find robocup_2025_description)/meshes/right_hipjoint_abd_1.stl" scale="0.001 0.001 0.001"/>
     </geometry>
     <material name="silver"/>
@@ -60,5 +60,5 @@
     <origin xyz="0.001764 0.041462 -0.380789" rpy="0 0 0"/>
     <geometry>
-      <mesh filename="file://$(find RCKO2025_description)/meshes/right_hipjoint_abd_1.stl" scale="0.001 0.001 0.001"/>
+      <mesh filename="file://$(find robocup_2025_description)/meshes/right_hipjoint_abd_1.stl" scale="0.001 0.001 0.001"/>
     </geometry>
   </collision>
@@ -73,5 +73,5 @@
     <origin xyz="0.042704 0.041484 -0.313789" rpy="0 0 0"/>
     <geometry>
-      <mesh filename="file://$(find RCKO2025_description)/meshes/right_hipjoint_pitch_1.stl" scale="0.001 0.001 0.001"/>
+      <mesh filename="file://$(find robocup_2025_description)/meshes/right_hipjoint_pitch_1.stl" scale="0.001 0.001 0.001"/>
     </geometry>
     <material name="silver"/>
@@ -80,5 +80,5 @@
     <origin xyz="0.042704 0.041484 -0.313789" rpy="0 0 0"/>
     <geometry>
-      <mesh filename="file://$(find RCKO2025_description)/meshes/right_hipjoint_pitch_1.stl" scale="0.001 0.001 0.001"/>
+      <mesh filename="file://$(find robocup_2025_description)/meshes/right_hipjoint_pitch_1.stl" scale="0.001 0.001 0.001"/>
     </geometry>
   </collision>
@@ -93,5 +93,5 @@
     <origin xyz="0.042204 -0.048516 -0.313759" rpy="0 0 0"/>
     <geometry>
-      <mesh filename="file://$(find RCKO2025_description)/meshes/left_hipjoint_pitch_1.stl" scale="0.001 0.001 0.001"/>
+      <mesh filename="file://$(find robocup_2025_description)/meshes/left_hipjoint_pitch_1.stl" scale="0.001 0.001 0.001"/>
     </geometry>
     <material name="silver"/>
@@ -100,5 +100,5 @@
     <origin xyz="0.042204 -0.048516 -0.313759" rpy="0 0 0"/>
     <geometry>
-      <mesh filename="file://$(find RCKO2025_description)/meshes/left_hipjoint_pitch_1.stl" scale="0.001 0.001 0.001"/>
+      <mesh filename="file://$(find robocup_2025_description)/meshes/left_hipjoint_pitch_1.stl" scale="0.001 0.001 0.001"/>
     </geometry>
   </collision>
@@ -113,5 +113,5 @@
     <origin xyz="0.002204 0.065525 -0.333776" rpy="0 0 0"/>
     <geometry>
-      <mesh filename="file://$(find RCKO2025_description)/meshes/right_upper_leg__1.stl" scale="0.001 0.001 0.001"/>
+      <mesh filename="file://$(find robocup_2025_description)/meshes/right_upper_leg__1.stl" scale="0.001 0.001 0.001"/>
     </geometry>
     <material name="silver"/>
@@ -120,5 +120,5 @@
     <origin xyz="0.002204 0.065525 -0.333776" rpy="0 0 0"/>
     <geometry>
-      <mesh filename="file://$(find RCKO2025_description)/meshes/right_upper_leg__1.stl" scale="0.001 0.001 0.001"/>
+      <mesh filename="file://$(find robocup_2025_description)/meshes/right_upper_leg__1.stl" scale="0.001 0.001 0.001"/>
     </geometry>
   </collision>
@@ -133,5 +133,5 @@
     <origin xyz="0.001704 -0.072749 -0.333513" rpy="0 0 0"/>
     <geometry>
-      <mesh filename="file://$(find RCKO2025_description)/meshes/left_upper_leg__1.stl" scale="0.001 0.001 0.001"/>
+      <mesh filename="file://$(find robocup_2025_description)/meshes/left_upper_leg__1.stl" scale="0.001 0.001 0.001"/>
     </geometry>
     <material name="silver"/>
@@ -140,9 +140,9 @@
     <origin xyz="0.001704 -0.072749 -0.333513" rpy="0 0 0"/>
     <geometry>
-      <mesh filename="file://$(find RCKO2025_description)/meshes/left_upper_leg__1.stl" scale="0.001 0.001 0.001"/>
-    </geometry>
-  </collision>
-</link>
-<link name="left_lower_leg_1">
+      <mesh filename="file://$(find robocup_2025_description)/meshes/left_upper_leg__1.stl" scale="0.001 0.001 0.001"/>
+    </geometry>
+  </collision>
+</link>
+<link name="right_lower_leg_1">
   <inertial>
     <origin xyz="-8.212056945443085e-05 0.02582198317065247 -0.06795536785927817" rpy="0 0 0"/>
@@ -153,5 +153,5 @@
     <origin xyz="0.002204 0.069395 -0.193786" rpy="0 0 0"/>
     <geometry>
-      <mesh filename="file://$(find RCKO2025_description)/meshes/left_lower_leg_1.stl" scale="0.001 0.001 0.001"/>
+      <mesh filename="file://$(find robocup_2025_description)/meshes/right_lower_leg_1.stl" scale="0.001 0.001 0.001"/>
     </geometry>
     <material name="silver"/>
@@ -160,9 +160,9 @@
     <origin xyz="0.002204 0.069395 -0.193786" rpy="0 0 0"/>
     <geometry>
-      <mesh filename="file://$(find RCKO2025_description)/meshes/left_lower_leg_1.stl" scale="0.001 0.001 0.001"/>
-    </geometry>
-  </collision>
-</link>
-<link name="right_lower_leg_1">
+      <mesh filename="file://$(find robocup_2025_description)/meshes/right_lower_leg_1.stl" scale="0.001 0.001 0.001"/>
+    </geometry>
+  </collision>
+</link>
+<link name="left_lower_leg_1">
   <inertial>
     <origin xyz="0.0005403758644121504 -0.02556694352281455 -0.0677062657730472" rpy="0 0 0"/>
@@ -173,5 +173,5 @@
     <origin xyz="0.003305 -0.075261 -0.193501" rpy="0 0 0"/>
     <geometry>
-      <mesh filename="file://$(find RCKO2025_description)/meshes/right_lower_leg_1.stl" scale="0.001 0.001 0.001"/>
+      <mesh filename="file://$(find robocup_2025_description)/meshes/left_lower_leg_1.stl" scale="0.001 0.001 0.001"/>
     </geometry>
     <material name="silver"/>
@@ -180,5 +180,5 @@
     <origin xyz="0.003305 -0.075261 -0.193501" rpy="0 0 0"/>
     <geometry>
-      <mesh filename="file://$(find RCKO2025_description)/meshes/right_lower_leg_1.stl" scale="0.001 0.001 0.001"/>
+      <mesh filename="file://$(find robocup_2025_description)/meshes/left_lower_leg_1.stl" scale="0.001 0.001 0.001"/>
     </geometry>
   </collision>
@@ -193,5 +193,5 @@
     <origin xyz="0.0018 -0.075186 -0.053506" rpy="0 0 0"/>
     <geometry>
-      <mesh filename="file://$(find RCKO2025_description)/meshes/left_ankle_pitch_1.stl" scale="0.001 0.001 0.001"/>
+      <mesh filename="file://$(find robocup_2025_description)/meshes/left_ankle_pitch_1.stl" scale="0.001 0.001 0.001"/>
     </geometry>
     <material name="silver"/>
@@ -200,5 +200,5 @@
     <origin xyz="0.0018 -0.075186 -0.053506" rpy="0 0 0"/>
     <geometry>
-      <mesh filename="file://$(find RCKO2025_description)/meshes/left_ankle_pitch_1.stl" scale="0.001 0.001 0.001"/>
+      <mesh filename="file://$(find robocup_2025_description)/meshes/left_ankle_pitch_1.stl" scale="0.001 0.001 0.001"/>
     </geometry>
   </collision>
@@ -213,5 +213,5 @@
     <origin xyz="0.001984 0.069765 -0.053787" rpy="0 0 0"/>
     <geometry>
-      <mesh filename="file://$(find RCKO2025_description)/meshes/right_ankle_pitch_1.stl" scale="0.001 0.001 0.001"/>
+      <mesh filename="file://$(find robocup_2025_description)/meshes/right_ankle_pitch_1.stl" scale="0.001 0.001 0.001"/>
     </geometry>
     <material name="silver"/>
@@ -220,5 +220,5 @@
     <origin xyz="0.001984 0.069765 -0.053787" rpy="0 0 0"/>
     <geometry>
-      <mesh filename="file://$(find RCKO2025_description)/meshes/right_ankle_pitch_1.stl" scale="0.001 0.001 0.001"/>
+      <mesh filename="file://$(find robocup_2025_description)/meshes/right_ankle_pitch_1.stl" scale="0.001 0.001 0.001"/>
     </geometry>
   </collision>
@@ -233,5 +233,5 @@
     <origin xyz="0.042277 0.045405 -0.07394" rpy="0 0 0"/>
     <geometry>
-      <mesh filename="file://$(find RCKO2025_description)/meshes/right_foot_1.stl" scale="0.001 0.001 0.001"/>
+      <mesh filename="file://$(find robocup_2025_description)/meshes/right_foot_1.stl" scale="0.001 0.001 0.001"/>
     </geometry>
     <material name="silver"/>
@@ -240,5 +240,5 @@
     <origin xyz="0.042277 0.045405 -0.07394" rpy="0 0 0"/>
     <geometry>
-      <mesh filename="file://$(find RCKO2025_description)/meshes/right_foot_1.stl" scale="0.001 0.001 0.001"/>
+      <mesh filename="file://$(find robocup_2025_description)/meshes/right_foot_1.stl" scale="0.001 0.001 0.001"/>
     </geometry>
   </collision>
@@ -253,5 +253,5 @@
     <origin xyz="0.042447 -0.051017 -0.073175" rpy="0 0 0"/>
     <geometry>
-      <mesh filename="file://$(find RCKO2025_description)/meshes/left_foot_1.stl" scale="0.001 0.001 0.001"/>
+      <mesh filename="file://$(find robocup_2025_description)/meshes/left_foot_1.stl" scale="0.001 0.001 0.001"/>
     </geometry>
     <material name="silver"/>
@@ -260,5 +260,5 @@
     <origin xyz="0.042447 -0.051017 -0.073175" rpy="0 0 0"/>
     <geometry>
-      <mesh filename="file://$(find RCKO2025_description)/meshes/left_foot_1.stl" scale="0.001 0.001 0.001"/>
+      <mesh filename="file://$(find robocup_2025_description)/meshes/left_foot_1.stl" scale="0.001 0.001 0.001"/>
     </geometry>
   </collision>
@@ -276,5 +276,5 @@
   <axis xyz="-0.0 -0.000326 -1.0"/>
 </joint>
-<joint name="rotate_10" type="continuous">
+<joint name="rotate_11" type="continuous">
   <origin xyz="-0.04094 -2.2e-05 -0.067" rpy="0 0 0"/>
   <parent link="right_hipjoint_abd_1"/>
@@ -282,5 +282,5 @@
   <axis xyz="1.0 0.0 0.0"/>
 </joint>
-<joint name="rotate_11" type="continuous">
+<joint name="rotate_10" type="continuous">
   <origin xyz="-0.04044 -2.2e-05 -0.067" rpy="0 0 0"/>
   <parent link="left_hipjoint_abd_1"/>
@@ -303,5 +303,5 @@
   <origin xyz="0.0 -0.00387 -0.13999" rpy="0 0 0"/>
   <parent link="right_upper_leg__1"/>
-  <child link="left_lower_leg_1"/>
+  <child link="right_lower_leg_1"/>
   <axis xyz="-0.0 -0.999997 0.002644"/>
 </joint>
@@ -309,10 +309,10 @@
   <origin xyz="-0.001601 0.002512 -0.140012" rpy="0 0 0"/>
   <parent link="left_upper_leg__1"/>
-  <child link="right_lower_leg_1"/>
+  <child link="left_lower_leg_1"/>
   <axis xyz="0.0 0.999975 -0.007053"/>
 </joint>
 <joint name="rotate_18" type="continuous">
   <origin xyz="0.001505 -7.5e-05 -0.139995" rpy="0 0 0"/>
-  <parent link="right_lower_leg_1"/>
+  <parent link="left_lower_leg_1"/>
   <child link="left_ankle_pitch_1"/>
   <axis xyz="-0.0 -0.999975 0.007053"/>
@@ -320,5 +320,5 @@
 <joint name="rotate_19" type="continuous">
   <origin xyz="0.00022 -0.00037 -0.139999" rpy="0 0 0"/>
-  <parent link="left_lower_leg_1"/>
+  <parent link="right_lower_leg_1"/>
   <child link="right_ankle_pitch_1"/>
   <axis xyz="0.0 0.999997 -0.002644"/>
