Commit message: EE dummy fix

File: humanoid_mani_description/urdf/humanoid_mani.xacro (robot description, xacro)
@@ -46,5 +46,5 @@
 <link name="eye_1">
   <inertial>
-    <origin xyz="5.505110954977244e-07 -4.6964214973910234e-07 0.00020929180740678066" rpy="0 0 0"/>
+    <origin xyz="5.505110955983383e-07 -4.696418934788116e-07 0.00020929180729237218" rpy="0 0 0"/>
     <mass value="1.902707681457099e-07"/>
     <inertia ixx="0.0" iyy="0.0" izz="0.0" ixy="0.0" iyz="0.0" ixz="0.0"/>
@@ -126,10 +126,10 @@
 <link name="ee_link_1">
   <inertial>
-    <origin xyz="-6.218104927793559e-07 1.652572509247552e-05 -0.00011133278533460855" rpy="0 0 0"/>
+    <origin xyz="0.26332737818950636 0.284305414795442 -0.09156863098650823" rpy="0 0 0"/>
     <mass value="1.9027076814554607e-07"/>
-    <inertia ixx="0.0" iyy="0.0" izz="0.0" ixy="0.0" iyz="-0.0" ixz="-0.0"/>
-  </inertial>
-  <visual>
-    <origin xyz="-0.002772 0.413548 -0.080544" rpy="0 0 0"/>
+    <inertia ixx="0.0" iyy="0.0" izz="0.0" ixy="-0.0" iyz="0.0" ixz="-0.0"/>
+  </inertial>
+  <visual>
+    <origin xyz="0.260556 0.717853 -0.172" rpy="0 0 0"/>
     <geometry>
       <mesh filename="file://$(find humanoid_mani_description)/meshes/ee_link_1.stl" scale="0.001 0.001 0.001"/>
@@ -138,5 +138,5 @@
   </visual>
   <collision>
-    <origin xyz="-0.002772 0.413548 -0.080544" rpy="0 0 0"/>
+    <origin xyz="0.260556 0.717853 -0.172" rpy="0 0 0"/>
     <geometry>
       <mesh filename="file://$(find humanoid_mani_description)/meshes/ee_link_1.stl" scale="0.001 0.001 0.001"/>
@@ -146,5 +146,5 @@
 <link name="Head_1">
   <inertial>
-    <origin xyz="-0.013469787584827716 -0.015314559330600433 0.03527216999851682" rpy="0 0 0"/>
+    <origin xyz="-0.013469787584827699 -0.015314559330375729 0.03527216999861435" rpy="0 0 0"/>
     <mass value="0.6173958690072822"/>
     <inertia ixx="0.00062" iyy="0.000263" izz="0.000484" ixy="-9e-06" iyz="-2.6e-05" ixz="-2.1e-05"/>
@@ -194,5 +194,5 @@
 </joint>
 <joint name="ee_dummy" type="fixed">
-  <origin xyz="0.0044 -0.144823 -0.020415" rpy="0 0 0"/>
+  <origin xyz="-0.258928 -0.449128 0.071041" rpy="0 0 0"/>
   <parent link="forearm_1"/>
   <child link="ee_link_1"/>
@@ -202,5 +202,5 @@
   <parent link="torso_1"/>
   <child link="Head_1"/>
-  <axis xyz="0.0 -1.0 -0.0"/>
+  <axis xyz="-0.0 1.0 0.0"/>
 </joint>
 </robot>

Commit message: 123

File: humanoid_mani_description/urdf/humanoid_mani.xacro (robot description, xacro)
@@ -6,7 +6,7 @@
 <link name="base_link">
   <inertial>
-    <origin xyz="0.00014449795003466327 6.165012944592263e-14 -0.002480473640778647" rpy="0 0 0"/>
+    <origin xyz="0.00014449791335857415 1.0295259413262148e-07 -0.0024804736407786827" rpy="0 0 0"/>
     <mass value="0.03383387831439711"/>
-    <inertia ixx="7e-06" iyy="7e-06" izz="1.4e-05" ixy="-0.0" iyz="0.0" ixz="0.0"/>
+    <inertia ixx="7e-06" iyy="7e-06" izz="1.4e-05" ixy="0.0" iyz="0.0" ixz="0.0"/>
   </inertial>
   <visual>
@@ -26,10 +26,10 @@
 <link name="torso_1">
   <inertial>
-    <origin xyz="-0.012877989784504057 -0.02595890872786548 0.09008175998722667" rpy="0 0 0"/>
+    <origin xyz="-0.012859491198833473 -0.025968077505632986 0.09008175998722645" rpy="0 0 0"/>
     <mass value="2.1937092001925604"/>
-    <inertia ixx="0.010947" iyy="0.008342" izz="0.007941" ixy="0.000264" iyz="0.000807" ixz="-0.001099"/>
-  </inertial>
-  <visual>
-    <origin xyz="-0.0 -0.0 -0.0" rpy="0 0 0"/>
+    <inertia ixx="0.010947" iyy="0.008343" izz="0.007941" ixy="0.000266" iyz="0.000807" ixz="-0.001099"/>
+  </inertial>
+  <visual>
+    <origin xyz="0.0 0.0 0.0" rpy="0 0 0"/>
     <geometry>
       <mesh filename="file://$(find humanoid_mani_description)/meshes/torso_1.stl" scale="0.001 0.001 0.001"/>
@@ -38,5 +38,5 @@
   </visual>
   <collision>
-    <origin xyz="-0.0 -0.0 -0.0" rpy="0 0 0"/>
+    <origin xyz="0.0 0.0 0.0" rpy="0 0 0"/>
     <geometry>
       <mesh filename="file://$(find humanoid_mani_description)/meshes/torso_1.stl" scale="0.001 0.001 0.001"/>
@@ -46,10 +46,10 @@
 <link name="eye_1">
   <inertial>
-    <origin xyz="5.505110955983383e-07 -4.696418934788116e-07 0.00020929180729237218" rpy="0 0 0"/>
+    <origin xyz="5.588157334333876e-07 3.6210216278198537e-07 0.00020929180729215013" rpy="0 0 0"/>
     <mass value="1.902707681457099e-07"/>
     <inertia ixx="0.0" iyy="0.0" izz="0.0" ixy="0.0" iyz="0.0" ixz="0.0"/>
   </inertial>
   <visual>
-    <origin xyz="-0.025041 -0.039279 -0.18636" rpy="0 0 0"/>
+    <origin xyz="-0.025013 -0.039296 -0.18636" rpy="0 0 0"/>
     <geometry>
       <mesh filename="file://$(find humanoid_mani_description)/meshes/eye_1.stl" scale="0.001 0.001 0.001"/>
@@ -58,5 +58,5 @@
   </visual>
   <collision>
-    <origin xyz="-0.025041 -0.039279 -0.18636" rpy="0 0 0"/>
+    <origin xyz="-0.025013 -0.039296 -0.18636" rpy="0 0 0"/>
     <geometry>
       <mesh filename="file://$(find humanoid_mani_description)/meshes/eye_1.stl" scale="0.001 0.001 0.001"/>
@@ -66,10 +66,10 @@
 <link name="shoulder_1">
   <inertial>
-    <origin xyz="-0.0008021063538195136 -0.01263269248673439 -0.002599544084532862" rpy="0 0 0"/>
+    <origin xyz="-0.0007928265132074144 -0.012632741596309643 -0.002599544084533001" rpy="0 0 0"/>
     <mass value="0.06721028329114603"/>
     <inertia ixx="1.7e-05" iyy="2.8e-05" izz="3.3e-05" ixy="-0.0" iyz="-3e-06" ixz="-0.0"/>
   </inertial>
   <visual>
-    <origin xyz="0.000708 0.093025 -0.10546" rpy="0 0 0"/>
+    <origin xyz="0.000642 0.093026 -0.10546" rpy="0 0 0"/>
     <geometry>
       <mesh filename="file://$(find humanoid_mani_description)/meshes/shoulder_1.stl" scale="0.001 0.001 0.001"/>
@@ -78,5 +78,5 @@
   </visual>
   <collision>
-    <origin xyz="0.000708 0.093025 -0.10546" rpy="0 0 0"/>
+    <origin xyz="0.000642 0.093026 -0.10546" rpy="0 0 0"/>
     <geometry>
       <mesh filename="file://$(find humanoid_mani_description)/meshes/shoulder_1.stl" scale="0.001 0.001 0.001"/>
@@ -86,10 +86,10 @@
 <link name="upperarm_1">
   <inertial>
-    <origin xyz="0.020532400219094592 -0.07168950541218574 -8.737550710166686e-06" rpy="0 0 0"/>
+    <origin xyz="0.02058391290540538 -0.07167462782007442 -8.737550710402608e-06" rpy="0 0 0"/>
     <mass value="0.7964005518324352"/>
-    <inertia ixx="0.002858" iyy="0.000163" izz="0.002858" ixy="2e-06" iyz="1e-06" ixz="0.0"/>
-  </inertial>
-  <visual>
-    <origin xyz="0.022178 0.125525 -0.08046" rpy="0 0 0"/>
+    <inertia ixx="0.002858" iyy="0.000163" izz="0.002858" ixy="4e-06" iyz="1e-06" ixz="-0.0"/>
+  </inertial>
+  <visual>
+    <origin xyz="0.022089 0.125541 -0.08046" rpy="0 0 0"/>
     <geometry>
       <mesh filename="file://$(find humanoid_mani_description)/meshes/upperarm_1.stl" scale="0.001 0.001 0.001"/>
@@ -98,5 +98,5 @@
   </visual>
   <collision>
-    <origin xyz="0.022178 0.125525 -0.08046" rpy="0 0 0"/>
+    <origin xyz="0.022089 0.125541 -0.08046" rpy="0 0 0"/>
     <geometry>
       <mesh filename="file://$(find humanoid_mani_description)/meshes/upperarm_1.stl" scale="0.001 0.001 0.001"/>
@@ -104,12 +104,32 @@
   </collision>
 </link>
+<link name="Head_1">
+  <inertial>
+    <origin xyz="-0.01345906594690515 -0.01532474151429016 0.03527216999861413" rpy="0 0 0"/>
+    <mass value="0.6173958690072822"/>
+    <inertia ixx="0.00062" iyy="0.000263" izz="0.000484" ixy="-8e-06" iyz="-2.6e-05" ixz="-2.1e-05"/>
+  </inertial>
+  <visual>
+    <origin xyz="-0.023026 -0.021333 -0.14636" rpy="0 0 0"/>
+    <geometry>
+      <mesh filename="file://$(find humanoid_mani_description)/meshes/Head_1.stl" scale="0.001 0.001 0.001"/>
+    </geometry>
+    <material name="silver"/>
+  </visual>
+  <collision>
+    <origin xyz="-0.023026 -0.021333 -0.14636" rpy="0 0 0"/>
+    <geometry>
+      <mesh filename="file://$(find humanoid_mani_description)/meshes/Head_1.stl" scale="0.001 0.001 0.001"/>
+    </geometry>
+  </collision>
+</link>
 <link name="forearm_1">
   <inertial>
-    <origin xyz="0.018319068322047685 -0.11944378738890721 -0.02034305937007909" rpy="0 0 0"/>
-    <mass value="1.088969578492718"/>
-    <inertia ixx="0.001507" iyy="0.000389" izz="0.001483" ixy="0.000207" iyz="-2e-06" ixz="3e-06"/>
-  </inertial>
-  <visual>
-    <origin xyz="0.001628 0.268725 -0.100959" rpy="0 0 0"/>
+    <origin xyz="0.01942621915712284 -0.1088730759389151 -0.020309797850417033" rpy="0 0 0"/>
+    <mass value="0.7439602672633931"/>
+    <inertia ixx="0.001136" iyy="0.000306" izz="0.001159" ixy="0.000233" iyz="-1e-06" ixz="3e-06"/>
+  </inertial>
+  <visual>
+    <origin xyz="0.001437 0.268726 -0.100959" rpy="0 0 0"/>
     <geometry>
       <mesh filename="file://$(find humanoid_mani_description)/meshes/forearm_1.stl" scale="0.001 0.001 0.001"/>
@@ -118,5 +138,5 @@
   </visual>
   <collision>
-    <origin xyz="0.001628 0.268725 -0.100959" rpy="0 0 0"/>
+    <origin xyz="0.001437 0.268726 -0.100959" rpy="0 0 0"/>
     <geometry>
       <mesh filename="file://$(find humanoid_mani_description)/meshes/forearm_1.stl" scale="0.001 0.001 0.001"/>
@@ -126,10 +146,10 @@
 <link name="ee_link_1">
   <inertial>
-    <origin xyz="0.26332737818950636 0.284305414795442 -0.09156863098650823" rpy="0 0 0"/>
-    <mass value="1.9027076814554607e-07"/>
-    <inertia ixx="0.0" iyy="0.0" izz="0.0" ixy="-0.0" iyz="0.0" ixz="-0.0"/>
-  </inertial>
-  <visual>
-    <origin xyz="0.260556 0.717853 -0.172" rpy="0 0 0"/>
+    <origin xyz="-7.265875284585485e-07 -4.978615931738872e-07 0.00020935007448756593" rpy="0 0 0"/>
+    <mass value="1.902707681457099e-07"/>
+    <inertia ixx="0.0" iyy="0.0" izz="0.0" ixy="0.0" iyz="0.0" ixz="0.0"/>
+  </inertial>
+  <visual>
+    <origin xyz="-0.003081 0.433545 -0.080544" rpy="0 0 0"/>
     <geometry>
       <mesh filename="file://$(find humanoid_mani_description)/meshes/ee_link_1.stl" scale="0.001 0.001 0.001"/>
@@ -138,27 +158,7 @@
   </visual>
   <collision>
-    <origin xyz="0.260556 0.717853 -0.172" rpy="0 0 0"/>
+    <origin xyz="-0.003081 0.433545 -0.080544" rpy="0 0 0"/>
     <geometry>
       <mesh filename="file://$(find humanoid_mani_description)/meshes/ee_link_1.stl" scale="0.001 0.001 0.001"/>
-    </geometry>
-  </collision>
-</link>
-<link name="Head_1">
-  <inertial>
-    <origin xyz="-0.013469787584827699 -0.015314559330375729 0.03527216999861435" rpy="0 0 0"/>
-    <mass value="0.6173958690072822"/>
-    <inertia ixx="0.00062" iyy="0.000263" izz="0.000484" ixy="-9e-06" iyz="-2.6e-05" ixz="-2.1e-05"/>
-  </inertial>
-  <visual>
-    <origin xyz="-0.023041 -0.021316 -0.14636" rpy="0 0 0"/>
-    <geometry>
-      <mesh filename="file://$(find humanoid_mani_description)/meshes/Head_1.stl" scale="0.001 0.001 0.001"/>
-    </geometry>
-    <material name="silver"/>
-  </visual>
-  <collision>
-    <origin xyz="-0.023041 -0.021316 -0.14636" rpy="0 0 0"/>
-    <geometry>
-      <mesh filename="file://$(find humanoid_mani_description)/meshes/Head_1.stl" scale="0.001 0.001 0.001"/>
     </geometry>
   </collision>
@@ -171,36 +171,36 @@
 </joint>
 <joint name="rgb_dummy" type="fixed">
-  <origin xyz="0.002 0.017963 0.04" rpy="0 0 0"/>
+  <origin xyz="0.001987 0.017963 0.04" rpy="0 0 0"/>
   <parent link="Head_1"/>
   <child link="eye_1"/>
 </joint>
 <joint name="rotate_1" type="continuous">
-  <origin xyz="-0.000708 -0.093025 0.10546" rpy="0 0 0"/>
+  <origin xyz="-0.000642 -0.093026 0.10546" rpy="0 0 0"/>
   <parent link="torso_1"/>
   <child link="shoulder_1"/>
-  <axis xyz="0.0 -1.0 -0.0"/>
+  <axis xyz="0.000712 -1.0 -0.0"/>
 </joint>
 <joint name="rotate_3" type="continuous">
-  <origin xyz="-0.02147 -0.0325 -0.025" rpy="0 0 0"/>
+  <origin xyz="-0.021447 -0.032515 -0.025" rpy="0 0 0"/>
   <parent link="shoulder_1"/>
   <child link="upperarm_1"/>
-  <axis xyz="1.0 -0.0 -0.0"/>
+  <axis xyz="1.0 0.000712 -0.0"/>
+</joint>
+<joint name="rotate_tilt" type="continuous">
+  <origin xyz="0.023026 0.021333 0.14636" rpy="0 0 0"/>
+  <parent link="torso_1"/>
+  <child link="Head_1"/>
+  <axis xyz="-0.000712 1.0 0.0"/>
 </joint>
 <joint name="rotate_5" type="continuous">
-  <origin xyz="0.02055 -0.1432 0.020499" rpy="0 0 0"/>
+  <origin xyz="0.020652 -0.143185 0.020499" rpy="0 0 0"/>
   <parent link="upperarm_1"/>
   <child link="forearm_1"/>
   <axis xyz="0.0 -7e-06 1.0"/>
 </joint>
-<joint name="ee_dummy" type="fixed">
-  <origin xyz="-0.258928 -0.449128 0.071041" rpy="0 0 0"/>
+<joint name="rigid_dummy" type="fixed">
+  <origin xyz="0.004518 -0.164819 -0.020415" rpy="0 0 0"/>
   <parent link="forearm_1"/>
   <child link="ee_link_1"/>
 </joint>
-<joint name="rotate_tilt" type="continuous">
-  <origin xyz="0.023041 0.021316 0.14636" rpy="0 0 0"/>
-  <parent link="torso_1"/>
-  <child link="Head_1"/>
-  <axis xyz="-0.0 1.0 0.0"/>
-</joint>
 </robot>

Commit message: joint cfg setup done

File: humanoid_mani_description/urdf/humanoid_mani.xacro (robot description, xacro)
@@ -164,9 +164,10 @@
   </collision>
 </link>
-<joint name="rotate_torso" type="continuous">
+<joint name="rotate_torso" type="revolute">
   <origin xyz="0.0 0.0 0.0" rpy="0 0 0"/>
   <parent link="base_link"/>
   <child link="torso_1"/>
   <axis xyz="0.0 -0.0 1.0"/>
+  <limit effort="100.0" lower="-3.1415" upper="3.1415" velocity="1.0"/>
 </joint>
 <joint name="rgb_dummy" type="fixed">
@@ -175,29 +176,33 @@
   <child link="eye_1"/>
 </joint>
-<joint name="rotate_1" type="continuous">
+<joint name="rotate_1" type="revolute">
   <origin xyz="-0.000642 -0.093026 0.10546" rpy="0 0 0"/>
   <parent link="torso_1"/>
   <child link="shoulder_1"/>
   <axis xyz="0.000712 -1.0 -0.0"/>
-</joint>
-<joint name="rotate_3" type="continuous">
-  <origin xyz="-0.021447 -0.032515 -0.025" rpy="0 0 0"/>
+  <limit effort="100.0" lower="-3.1415" upper="3.1415" velocity="1.0"/>
+</joint>
+<joint name="rotate_3" type="revolute">
+  <origin xyz="-0.021447 -0.032515 -0.025" rpy="1.5708 0 0"/>
   <parent link="shoulder_1"/>
   <child link="upperarm_1"/>
-  <axis xyz="1.0 0.000712 -0.0"/>
-</joint>
-<joint name="rotate_tilt" type="continuous">
+  <axis xyz="-1.0 0.0 0.0"/>
+  <limit effort="100.0" lower="-1.5708" upper="1.5708" velocity="1.0"/>
+</joint>
+<joint name="rotate_tilt" type="revolute">
   <origin xyz="0.023026 0.021333 0.14636" rpy="0 0 0"/>
   <parent link="torso_1"/>
   <child link="Head_1"/>
   <axis xyz="-0.000712 1.0 0.0"/>
-</joint>
-<joint name="rotate_5" type="continuous">
+  <limit effort="100.0" lower="0.0" upper="2.225" velocity="1.0"/>
+</joint>
+<joint name="rotate_5" type="revolute">
   <origin xyz="0.020652 -0.143185 0.020499" rpy="0 0 0"/>
   <parent link="upperarm_1"/>
   <child link="forearm_1"/>
   <axis xyz="0.0 -7e-06 1.0"/>
-</joint>
-<joint name="rigid_dummy" type="fixed">
+  <limit effort="100.0" lower="-2.462" upper="2.4" velocity="1.0"/>
+</joint>
+<joint name="ee_dummy" type="fixed">
   <origin xyz="0.004518 -0.164819 -0.020415" rpy="0 0 0"/>
   <parent link="forearm_1"/>
